File: Hardware/digichiver.kicad_sch (KiCad schematic)
At the start: 0 parts

Commit message: fix kicad project hierarchy
Other:
- added sheet Control (Control.kicad_sch)
- added sheet Digitalker (Digitalker.kicad_sch)
- added sheet Power (Power.kicad_sch)
Changed lines of the file:
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@@
 		(company "J. Thweatt")
+	)
+	(sheet
+		(at 194.31 107.95)
+		(size 19.05 16.51)
+		(exclude_from_sim no)
+		(in_bom yes)
+		(on_board yes)
+		(dnp no)
+		(fields_autoplaced yes)
+		(stroke
+			(width 0.1524)
+			(type solid)
+		)
+		(fill
+			(color 0 0 0 0)
+		)
+		(property "Sheetname" "Power"
+			(at 194.31 107.2384 0)
+			(show_name no)
+			(do_not_autoplace no)
+			(effects
+				(font
+					(size 1.27 1.27)
+				)
+				(justify left bottom)
+			)
+		)
+		(property "Sheetfile" "Power.kicad_sch"
+			(at 194.31 125.0446 0)
+			(show_name no)
+			(do_not_autoplace no)
+			(effects
+				(font
+					(size 1.27 1.27)
+				)
+				(justify left top)
+			)
+		)
+		(instances
+			(project "Digichiver"
+				(path "/51de4045-d2a2-42d9-b145-319acd726bb6"
+					(page "3")
+				)
+			)
+		)
+	)
+	(sheet
+		(at 240.03 87.63)
+		(size 27.94 21.59)
+		(exclude_from_sim no)
+		(in_bom yes)
+		(on_board yes)
+		(dnp no)
+		(fields_autoplaced yes)
+		(stroke
+			(width 0.1524)
+			(type solid)
+		)
+		(fill
+			(color 0 0 0 0)
+		)
+		(property "Sheetname" "Control"
+			(at 240.03 86.9184 0)
+			(show_name no)
+			(do_not_autoplace no)
+			(effects
+				(font
+					(size 1.27 1.27)
+				)
+				(justify left bottom)
+			)
+		)
+		(property "Sheetfile" "Control.kicad_sch"
+			(at 240.03 109.8046 0)
+			(show_name no)
+			(do_not_autoplace no)
+			(effects
+				(font
+					(size 1.27 1.27)
+				)
+				(justify left top)
+			)
+		)
+		(instances
+			(project "Digichiver"
+				(path "/51de4045-d2a2-42d9-b145-319acd726bb6"
+					(page "2")
+				)
+			)
+		)
+	)
+	(sheet
+		(at 140.97 148.59)
+		(size 33.02 27.94)
+		(exclude_from_sim no)
+		(in_bom yes)
+		(on_board yes)
+		(dnp no)
+		(fields_autoplaced yes)
+		(stroke
+			(width 0.1524)
+			(type solid)
+		)
+		(fill
+			(color 0 0 0 0)
+		)
+		(property "Sheetname" "Digitalker"
+			(at 140.97 147.8784 0)
+			(show_name no)
+			(do_not_autoplace no)
+			(effects
+				(font
+					(size 1.27 1.27)
+				)
+				(justify left bottom)
+			)
+		)
+		(property "Sheetfile" "Digitalker.kicad_sch"
+			(at 140.97 177.1146 0)
+			(show_name no)
+			(do_not_autoplace no)
+			(effects
+				(font
+					(size 1.27 1.27)
+				)
+				(justify left top)
+			)
+		)
+		(instances
+			(project "Digichiver"
+				(path "/51de4045-d2a2-42d9-b145-319acd726bb6"
+					(page "4")
+				)
+			)
+		)
 	)
 	(sheet_instances

Commit message: finish digitalker
Other:
- sheet Digitalker ports: added DIGITALKER_CLK_4MHZ, DIGITALKER_CMS, INTR, RDATA[0..7], ROM_ADDR[0..13], SW[1..8], ~{DIGITALKER_CS}, ~{DIGITALKER_WR}, ~{ROMEN}; removed none
Changed lines of the file:
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@@
 	)
 	(sheet
-		(at 194.31 107.95)
+		(at 127 152.4)
 		(size 19.05 16.51)
 		(exclude_from_sim no)
@@
 		)
 		(property "Sheetname" "Power"
-			(at 194.31 107.2384 0)
+			(at 127 151.6884 0)
 			(show_name no)
 			(do_not_autoplace no)
@@
 		)
 		(property "Sheetfile" "Power.kicad_sch"
-			(at 194.31 125.0446 0)
+			(at 127 169.4946 0)
 			(show_name no)
 			(do_not_autoplace no)
@@
 	)
 	(sheet
-		(at 240.03 87.63)
+		(at 201.93 101.6)
 		(size 27.94 21.59)
 		(exclude_from_sim no)
@@
 		)
 		(property "Sheetname" "Control"
-			(at 240.03 86.9184 0)
+			(at 201.93 100.8884 0)
 			(show_name no)
 			(do_not_autoplace no)
@@
 		)
 		(property "Sheetfile" "Control.kicad_sch"
-			(at 240.03 109.8046 0)
+			(at 201.93 123.7746 0)
 			(show_name no)
 			(do_not_autoplace no)
@@
 	)
 	(sheet
-		(at 140.97 148.59)
-		(size 33.02 27.94)
+		(at 279.4 124.46)
+		(size 38.1 25.4)
 		(exclude_from_sim no)
 		(in_bom yes)
@@
 		)
 		(property "Sheetname" "Digitalker"
-			(at 140.97 147.8784 0)
+			(at 279.4 123.7484 0)
 			(show_name no)
 			(do_not_autoplace no)
@@
 		)
 		(property "Sheetfile" "Digitalker.kicad_sch"
-			(at 140.97 177.1146 0)
+			(at 279.4 150.4446 0)
 			(show_name no)
 			(do_not_autoplace no)
@@
 			)
 		)
+		(pin "ROM_ADDR[0..13]" output
+			(at 317.5 127 0)
+			(effects
+				(font
+					(size 1.27 1.27)
+				)
+				(justify right)
+			)
+		)
+		(pin "RDATA[0..7]" input
+			(at 279.4 142.24 180)
+			(effects
+				(font
+					(size 1.27 1.27)
+				)
+				(justify left)
+			)
+		)
+		(pin "SW[1..8]" input
+			(at 279.4 137.16 180)
+			(effects
+				(font
+					(size 1.27 1.27)
+				)
+				(justify left)
+			)
+		)
+		(pin "~{DIGITALKER_WR}" input
+			(at 279.4 129.54 180)
+			(effects
+				(font
+					(size 1.27 1.27)
+				)
+				(justify left)
+			)
+		)
+		(pin "INTR" output
+			(at 317.5 147.32 0)
+			(effects
+				(font
+					(size 1.27 1.27)
+				)
+				(justify right)
+			)
+		)
+		(pin "DIGITALKER_CMS" input
+			(at 279.4 127 180)
+			(effects
+				(font
+					(size 1.27 1.27)
+				)
+				(justify left)
+			)
+		)
+		(pin "~{DIGITALKER_CS}" input
+			(at 279.4 132.08 180)
+			(effects
+				(font
+					(size 1.27 1.27)
+				)
+				(justify left)
+			)
+		)
+		(pin "DIGITALKER_CLK_4MHZ" input
+			(at 279.4 147.32 180)
+			(effects
+				(font
+					(size 1.27 1.27)
+				)
+				(justify left)
+			)
+		)
+		(pin "~{ROMEN}" output
+			(at 317.5 137.16 0)
+			(effects
+				(font
+					(size 1.27 1.27)
+				)
+				(justify right)
+			)
+		)

Commit message: power
Changed lines of the file:
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@@
 	)
 	(sheet
-		(at 127 152.4)
-		(size 19.05 16.51)
+		(at 207.01 189.23)
+		(size 38.1 16.51)
 		(exclude_from_sim no)
 		(in_bom yes)
@@
 		)
 		(property "Sheetname" "Power"
-			(at 127 151.6884 0)
+			(at 207.01 188.5184 0)
 			(show_name no)
 			(do_not_autoplace no)
@@
 		)
 		(property "Sheetfile" "Power.kicad_sch"
-			(at 127 169.4946 0)
+			(at 207.01 206.3246 0)
 			(show_name no)
 			(do_not_autoplace no)

Commit message: sync
Parts:
- added J2: USB_C_Receptacle, symbol Connector:USB_C_Receptacle
- added R19, R20: 5.1k, symbol Device:R_US
Connections:
- new net: J2.A5 (CC1), R19.2
- new net: J2.B5 (CC2), R20.2
- new net +5V: J2.A4 (VBUS), J2.A9 (VBUS), J2.B4 (VBUS), J2.B9 (VBUS)
- new net GND: J2.A1 (GND), J2.A12 (GND), J2.B1 (GND), J2.B12 (GND), J2.SH (SHIELD), R19.1, R20.1
- new net USB_D+: J2.A6 (D+), J2.B6 (D+)
- new net USB_D-: J2.A7 (D-), J2.B7 (D-)
- no-connect marks 0 -> 10
Other:
- sheet Control ports: added BCLK, DIGITALKER_CLK_4MHZ, DIGITALKER_CMS, FSYNC, INTR, RDATA[0..7], ROM_ADDR[0..13], SDATA, SW[1..8], USB_D+, USB_D-, ~{DIGITALKER_CS}, ~{DIGITALKER_WR}, ~{ROMEN}; removed none
