File: Hardware/digichiver.kicad_sch (KiCad schematic)
At the start: 3 parts, among them J2 USB_C_Receptacle

Commit message: implement PCM1809
Other:
- added sheet Audio (Audio.kicad_sch)
Changed lines of the file:
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@@
+		)
+	)
+	(sheet
+		(at 241.3 154.94)
+		(size 38.1 12.7)
+		(exclude_from_sim no)
+		(in_bom yes)
+		(on_board yes)
+		(dnp no)
+		(fields_autoplaced yes)
+		(stroke
+			(width 0.1524)
+			(type solid)
+		)
+		(fill
+			(color 0 0 0 0)
+		)
+		(property "Sheetname" "Audio"
+			(at 241.3 154.2284 0)
+			(show_name no)
+			(do_not_autoplace no)
+			(effects
+				(font
+					(size 1.27 1.27)
+				)
+				(justify left bottom)
+			)
+		)
+		(property "Sheetfile" "Audio.kicad_sch"
+			(at 241.3 168.2246 0)
+			(show_name no)
+			(do_not_autoplace no)
+			(effects
+				(font
+					(size 1.27 1.27)
+				)
+				(justify left top)
+			)
+		)
+		(instances
+			(project "digichiver"
+				(path "/51de4045-d2a2-42d9-b145-319acd726bb6"
+					(page "5")
+				)
+			)
 		)
 	)
