File: Hardware/Digichiver.kicad_sch (KiCad schematic)
At the start: 3 parts, among them J2 USB_C_Receptacle

Commit message: file renaming
Other:
- sheet Audio ports: added BCLK, FILTERED_SPEECH, FSYNC, SDATA; removed none
- sheet Digitalker ports: added FILTERED_SPEECH; removed none
Changed lines of the file:
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@@
+	(wire
+		(pts
+			(xy 283.21 156.21) (xy 279.4 156.21)
+		)
+		(stroke
+			(width 0)
+			(type default)
+		)
+	)
 	(wire
 		(pts
@@
 		)
 	)
+	(wire
+		(pts
+			(xy 203.2 158.75) (xy 241.3 158.75)
+		)
+		(stroke
+			(width 0)
+			(type default)
+		)
+	)
 	(bus
 		(pts
@@
 	(wire
 		(pts
+			(xy 203.2 161.29) (xy 241.3 161.29)
+		)
+		(stroke
+			(width 0)
+			(type default)
+		)
+	)
+	(wire
+		(pts
 			(xy 121.92 120.65) (xy 123.19 120.65)
 		)
@@
 	(wire
 		(pts
+			(xy 279.4 144.78) (xy 283.21 144.78)
+		)
+		(stroke
+			(width 0)
+			(type default)
+		)
+	)
+	(wire
+		(pts
 			(xy 123.19 125.73) (xy 165.1 125.73)
 		)
@@
 	(wire
 		(pts
+			(xy 283.21 144.78) (xy 283.21 156.21)
+		)
+		(stroke
+			(width 0)
+			(type default)
+		)
+	)
+	(wire
+		(pts
 			(xy 129.54 113.03) (xy 121.92 113.03)
 		)
@@
 		(pts
 			(xy 148.59 111.76) (xy 148.59 109.22)
+		)
+		(stroke
+			(width 0)
+			(type default)
+		)
+	)
+	(wire
+		(pts
+			(xy 203.2 156.21) (xy 241.3 156.21)
 		)
 		(stroke
@@
 		)
 		(instances
-			(project "digichiver"
+			(project "Digichiver"
 				(path "/51de4045-d2a2-42d9-b145-319acd726bb6"
 					(reference "#PWR071")
@@
 		)
 		(instances
-			(project "digichiver"
+			(project "Digichiver"
 				(path "/51de4045-d2a2-42d9-b145-319acd726bb6"
 					(reference "R19")
@@
 		)
 		(instances
-			(project "digichiver"
+			(project "Digichiver"
 				(path "/51de4045-d2a2-42d9-b145-319acd726bb6"
 					(reference "#PWR072")
@@
 		)
 		(instances
-			(project "digichiver"
+			(project "Digichiver"
 				(path "/51de4045-d2a2-42d9-b145-319acd726bb6"
 					(reference "#PWR034")
@@
 		)
 		(instances
-			(project "digichiver"
+			(project "Digichiver"
 				(path "/51de4045-d2a2-42d9-b145-319acd726bb6"
 					(reference "J2")
@@
 		)
 		(instances
-			(project "digichiver"
+			(project "Digichiver"
 				(path "/51de4045-d2a2-42d9-b145-319acd726bb6"
 					(reference "R20")
@@
 	)
 	(sheet
-		(at 165.1 167.64)
+		(at 165.1 171.45)
 		(size 38.1 16.51)
 		(exclude_from_sim no)
@@
 		)
 		(property "Sheetname" "Power"
-			(at 165.1 166.9284 0)
+			(at 165.1 170.7384 0)
 			(show_name no)
 			(do_not_autoplace no)
@@
 		)
 		(property "Sheetfile" "Power.kicad_sch"
-			(at 165.1 184.7346 0)
+			(at 165.1 188.5446 0)
 			(show_name no)
 			(do_not_autoplace no)
@@
 		)
 		(instances
-			(project "digichiver"
+			(project "Digichiver"
 				(path "/51de4045-d2a2-42d9-b145-319acd726bb6"
 					(page "3")
@@
 	(sheet
 		(at 165.1 118.11)
-		(size 38.1 43.18)
+		(size 38.1 45.72)
 		(exclude_from_sim no)
 		(in_bom yes)
@@
 		)
 		(property "Sheetfile" "Control.kicad_sch"
-			(at 165.1 161.8746 0)
+			(at 165.1 164.4146 0)
 			(show_name no)
 			(do_not_autoplace no)
@@
 		)
 		(pin "SDATA" input
-			(at 203.2 152.4 0)
+			(at 203.2 156.21 0)
 			(effects
 				(font
@@
 		)
 		(pin "BCLK" output
-			(at 203.2 154.94 0)
+			(at 203.2 158.75 0)
 			(effects
 				(font
@@
 		)
 		(pin "FSYNC" output
-			(at 203.2 157.48 0)
+			(at 203.2 161.29 0)
 			(effects
 				(font
@@
 		)
 		(instances
-			(project "digichiver"
+			(project "Digichiver"
 				(path "/51de4045-d2a2-42d9-b145-319acd726bb6"
 					(page "2")
@@
 			)
 		)
+		(pin "FILTERED_SPEECH" output
+			(at 279.4 144.78 0)
+			(effects
+				(font
+					(size 1.27 1.27)
+				)
+				(justify right)
+			)
+		)
 		(instances
-			(project "digichiver"
+			(project "Digichiver"
 				(path "/51de4045-d2a2-42d9-b145-319acd726bb6"
 					(page "4")
@@
 	)
 	(sheet
-		(at 241.3 154.94)
-		(size 38.1 12.7)
+		(at 241.3 153.67)
+		(size 38.1 10.16)
 		(exclude_from_sim no)
 		(in_bom yes)
@@
 		)
 		(property "Sheetname" "Audio"
-			(at 241.3 154.2284 0)
+			(at 241.3 152.9584 0)
 			(show_name no)
 			(do_not_autoplace no)
@@
 		)
 		(property "Sheetfile" "Audio.kicad_sch"
-			(at 241.3 168.2246 0)
+			(at 241.3 164.4146 0)
 			(show_name no)
 			(do_not_autoplace no)
@@
 			)
 		)
+		(pin "BCLK" input
+			(at 241.3 158.75 180)
+			(effects
+				(font
+					(size 1.27 1.27)
+				)
+				(justify left)
+			)
+		)
+		(pin "FILTERED_SPEECH" input
+			(at 279.4 156.21 0)
+			(effects
+				(font
+					(size 1.27 1.27)
+				)
+				(justify right)
+			)
+		)
+		(pin "FSYNC" input
+			(at 241.3 161.29 180)
+			(effects
+				(font
+					(size 1.27 1.27)
+				)
+				(justify left)
+			)
+		)
+		(pin "SDATA" output
+			(at 241.3 156.21 180)
+			(effects
+				(font
+					(size 1.27 1.27)
+				)
+				(justify left)
+			)
+		)
 		(instances
-			(project "digichiver"
+			(project "Digichiver"
 				(path "/51de4045-d2a2-42d9-b145-319acd726bb6"
 					(page "5")
