File: Hardware/Digichiver.kicad_sch (KiCad schematic)
At the start: 3 parts, among them J2 USB4105-GF-A

Commit message: rev2
move all components to top side and update BOM to use basic JLCPCB components when possible
Parts:
- R19, R20: JLCPCB Part # C105872 -> C25905; MPN RC0402FR-075K1L -> 0402WGF5101TCE
Changed lines of the file:
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@@
 	(title_block
 		(title "Digichiver")
-		(date "2026-07-24")
-		(rev "1")
+		(date "2026-09-01")
+		(rev "2")
 		(company "J. Thweatt")
 	)
@@
 			)
 		)
-		(property "MPN" "RC0402FR-075K1L"
+		(property "MPN" "0402WGF5101TCE"
 			(at 139.7 109.22 90)
 			(hide yes)
@@
 			)
 		)
-		(property "JLCPCB Part #" "C105872"
+		(property "JLCPCB Part #" "C25905"
 			(at 139.7 109.22 90)
 			(hide yes)
@@
 			)
 		)
-		(property "MPN" "RC0402FR-075K1L"
+		(property "MPN" "0402WGF5101TCE"
 			(at 139.7 111.76 90)
 			(hide yes)
@@
 			)
 		)
-		(property "JLCPCB Part #" "C105872"
+		(property "JLCPCB Part #" "C25905"
 			(at 139.7 111.76 90)
 			(hide yes)
