File: Hardware/Digitalker.kicad_sch (KiCad schematic)
At the start: 35 parts, among them U10 TLV9004IPWR, U2 SN74LVC245A, U3 SN74LVC245A, U4 SN74LVC8T245, U5 SN74LVC8T245, U6 SN74LVC8T245, X1 ICSockets-40P

Commit message: layout complete
Parts:
- renumbered X1 to XC1
Changed lines of the file:
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@@
 		(in_pos_files yes)
 		(dnp no)
-		(property "Reference" "X1"
+		(property "Reference" "XC1"
 			(at 203.2 88.138 0)
 			(show_name no)
@@
 			(project "Digichiver"
 				(path "/51de4045-d2a2-42d9-b145-319acd726bb6/ca4885d7-9004-4a4f-ae69-fc7e29c6fa33"
-					(reference "X1")
+					(reference "XC1")
 					(unit 1)
 				)
