File: Hardware/Digitalker.kicad_sch (KiCad schematic)
At the start: 35 parts, among them U10 TLV9004IPWR, U2 SN74LVC245A, U3 SN74LVC245A, U4 SN74LVC8T245, U5 SN74LVC8T245, U6 SN74LVC8T245

Commit message: generate outputs
Parts:
- C1, C2, C4, C42, C45, C46, C47, C5, C6, C7, C8, C9: JLCPCB Part # (none) -> C105883; MPN GRM155R71A104KA01D -> CC0402KRX7R8BB104; Voltage 10V -> 25V
- C3: JLCPCB Part # (none) -> C105883
- C41: JLCPCB Part # (none) -> C52923
- C43, C44: JLCPCB Part # (none) -> C5137480
- R1, R2, R3, R4, R5: JLCPCB Part # (none) -> C60490
- R21, R22, R23: JLCPCB Part # (none) -> C60491
- R24, R25: JLCPCB Part # (none) -> C163447
- R26, R27: JLCPCB Part # (none) -> C852943
- U10: JLCPCB Part # (none) -> C2058050; MPN TLV9004IPW -> TLV9004IPWR
- U2, U3: JLCPCB Part # (none) -> C7848; MPN SN74LVC245APW -> SN74LVC245APWR
- U4, U5, U6: JLCPCB Part # (none) -> C27643; MPN SN74LVC8T245PW -> SN74LVC8T245PWR
- XC1: JLCPCB Part # (none) -> C2332
