File: Hardware/Digitalker.kicad_sch (KiCad schematic)
At the start: 35 parts, among them U10 TLV9004IPWR, U2 SN74LVC245A, U3 SN74LVC245A, U4 SN74LVC8T245, U5 SN74LVC8T245, U6 SN74LVC8T245

Commit message: fix SN74LVC8T245 footprint
Parts:
- U4, U5, U6: footprint Package_SO:TSSOP-24_4.4x6.5mm_P0.5mm -> Package_SO:TSSOP-24_4.4x7.8mm_P0.65mm
Changed lines of the file:
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@@
 			)
 		)
-		(property "Footprint" "Package_SO:TSSOP-24_4.4x6.5mm_P0.5mm"
+		(property "Footprint" "Package_SO:TSSOP-24_4.4x7.8mm_P0.65mm"
 			(at 135.89 93.98 0)
 			(hide yes)
@@
 			)
 		)
-		(property "Footprint" "Package_SO:TSSOP-24_4.4x6.5mm_P0.5mm"
+		(property "Footprint" "Package_SO:TSSOP-24_4.4x7.8mm_P0.65mm"
 			(at 135.89 160.02 0)
 			(hide yes)
@@
 			)
 		)
-		(property "Footprint" "Package_SO:TSSOP-24_4.4x6.5mm_P0.5mm"
+		(property "Footprint" "Package_SO:TSSOP-24_4.4x7.8mm_P0.65mm"
 			(at 135.89 226.06 0)
 			(hide yes)

Commit message: rev2
move all components to top side and update BOM to use basic JLCPCB components when possible
Parts:
- C1, C2, C3, C4, C42, C45, C46, C47, C5, C6, C7, C8, C9: JLCPCB Part # C105883 -> C307331; MPN CC0402KRX7R8BB104 -> CL05B104KB54PNC
- C43, C44: JLCPCB Part # C5137480 -> C15195; Voltage 10V -> 50V
- R1, R2, R3, R4, R5: JLCPCB Part # C60490 -> C25744; MPN RC0402FR-0710KL -> 0402WGF1002TCE
- R21, R22, R23: JLCPCB Part # C60491 -> C25741; MPN RC0402FR-07100KL -> 0402WGF1003TCE
- R24, R25: JLCPCB Part # C163447 -> C25879; MPN RC0402JR-072K2L -> 0402WGF2201TCE
- R26, R27: JLCPCB Part # C852943 -> C25924; MPN RT0402BRD078K2L -> 0402WGF8201TCE
- XC1: now left out of the parts list
Changed lines of the file:
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@@
 	(title_block
 		(title "Digichiver")
-		(date "2026-07-24")
-		(rev "1")
+		(date "2026-09-01")
+		(rev "2")
 		(company "J. Thweatt")
 	)
@@
 			)
 		)
-		(property "MPN" "CC0402KRX7R8BB104"
+		(property "MPN" "CL05B104KB54PNC"
 			(at 119.38 106.68 0)
 			(hide yes)
@@
 			)
 		)
-		(property "JLCPCB Part #" "C105883"
+		(property "JLCPCB Part #" "C307331"
 			(at 119.38 106.68 0)
 			(hide yes)
@@
 			)
 		)
-		(property "MPN" "RC0402FR-07100KL"
+		(property "MPN" "0402WGF1003TCE"
 			(at 283.21 163.83 0)
 			(hide yes)
@@
 			)
 		)
-		(property "JLCPCB Part #" "C60491"
+		(property "JLCPCB Part #" "C25741"
 			(at 283.21 163.83 0)
 			(hide yes)
@@
 			)
 		)
-		(property "MPN" "RC0402FR-0710KL"
+		(property "MPN" "0402WGF1002TCE"
 			(at 281.94 111.76 0)
 			(hide yes)
@@
 			)
 		)
-		(property "JLCPCB Part #" "C60490"
+		(property "JLCPCB Part #" "C25744"
 			(at 281.94 111.76 0)
 			(hide yes)
@@
 			)
 		)
-		(property "MPN" "CC0402KRX7R8BB104"
+		(property "MPN" "CL05B104KB54PNC"
 			(at 226.06 81.28 90)
 			(hide yes)
@@
 			)
 		)
-		(property "JLCPCB Part #" "C105883"
+		(property "JLCPCB Part #" "C307331"
 			(at 226.06 81.28 90)
 			(hide yes)
@@
 			)
 		)
-		(property "MPN" "CC0402KRX7R8BB104"
+		(property "MPN" "CL05B104KB54PNC"
 			(at 111.76 172.72 0)
 			(hide yes)
@@
 			)
 		)
-		(property "JLCPCB Part #" "C105883"
+		(property "JLCPCB Part #" "C307331"
 			(at 111.76 172.72 0)
 			(hide yes)
@@
 			)
 		)
-		(property "MPN" "CC0402KRX7R8BB104"
+		(property "MPN" "CL05B104KB54PNC"
 			(at 111.76 40.64 0)
 			(hide yes)
@@
 			)
 		)
-		(property "JLCPCB Part #" "C105883"
+		(property "JLCPCB Part #" "C307331"
 			(at 111.76 40.64 0)
 			(hide yes)
@@
 			)
 		)
-		(property "MPN" "CC0402KRX7R8BB104"
+		(property "MPN" "CL05B104KB54PNC"
 			(at 336.55 175.26 90)
 			(hide yes)
@@
 			)
 		)
-		(property "JLCPCB Part #" "C105883"
+		(property "JLCPCB Part #" "C307331"
 			(at 336.55 175.26 90)
 			(hide yes)
@@
 			)
 		)
-		(property "MPN" "CC0402KRX7R8BB104"
+		(property "MPN" "CL05B104KB54PNC"
 			(at 119.38 40.64 0)
 			(hide yes)
@@
 			)
 		)
-		(property "JLCPCB Part #" "C105883"
+		(property "JLCPCB Part #" "C307331"
 			(at 119.38 40.64 0)
 			(hide yes)
@@
 			)
 		)
-		(property "MPN" "RC0402JR-072K2L"
+		(property "MPN" "0402WGF2201TCE"
 			(at 233.68 219.71 90)
 			(hide yes)
@@
 			)
 		)
-		(property "JLCPCB Part #" "C163447"
+		(property "JLCPCB Part #" "C25879"
 			(at 233.68 219.71 90)
 			(hide yes)
@@
 			)
 		)
-		(property "MPN" "RC0402JR-072K2L"
+		(property "MPN" "0402WGF2201TCE"
 			(at 220.98 219.71 90)
 			(hide yes)
@@
 			)
 		)
-		(property "JLCPCB Part #" "C163447"
+		(property "JLCPCB Part #" "C25879"
 			(at 220.98 219.71 90)
 			(hide yes)
@@
 			)
 		)
-		(property "MPN" "RC0402FR-0710KL"
+		(property "MPN" "0402WGF1002TCE"
 			(at 281.94 62.23 0)
 			(hide yes)
@@
 			)
 		)
-		(property "JLCPCB Part #" "C60490"
+		(property "JLCPCB Part #" "C25744"
 			(at 281.94 62.23 0)
 			(hide yes)
@@
 			)
 		)
-		(property "Voltage" "10V"
+		(property "Voltage" "50V"
 			(at 251.46 196.342 90)
 			(show_name no)
@@
 			)
 		)
-		(property "JLCPCB Part #" "C5137480"
+		(property "JLCPCB Part #" "C15195"
 			(at 251.46 199.39 90)
 			(hide yes)
@@
 			)
 		)
-		(property "MPN" "CC0402KRX7R8BB104"
+		(property "MPN" "CL05B104KB54PNC"
 			(at 269.24 157.48 0)
 			(hide yes)
@@
 			)
 		)
-		(property "JLCPCB Part #" "C105883"
+		(property "JLCPCB Part #" "C307331"
 			(at 269.24 157.48 0)
 			(hide yes)
@@
 			)
 		)
-		(property "MPN" "RC0402FR-07100KL"
+		(property "MPN" "0402WGF1003TCE"
 			(at 261.62 147.32 0)
 			(hide yes)
@@
 			)
 		)
-		(property "JLCPCB Part #" "C60491"
+		(property "JLCPCB Part #" "C25741"
 			(at 261.62 147.32 0)
 			(hide yes)
@@
 			)
 		)
-		(property "MPN" "RC0402FR-07100KL"
+		(property "MPN" "0402WGF1003TCE"
 			(at 261.62 157.48 0)
 			(hide yes)
@@
 			)
 		)
-		(property "JLCPCB Part #" "C60491"
+		(property "JLCPCB Part #" "C25741"
 			(at 261.62 157.48 0)
 			(hide yes)
@@
 			)
 		)
-		(property "MPN" "CC0402KRX7R8BB104"
+		(property "MPN" "CL05B104KB54PNC"
 			(at 111.76 106.68 0)
 			(hide yes)
@@
 			)
 		)
-		(property "JLCPCB Part #" "C105883"
+		(property "JLCPCB Part #" "C307331"
 			(at 111.76 106.68 0)
 			(hide yes)
@@
 			)
 		)
-		(property "MPN" "CC0402KRX7R8BB104"
+		(property "MPN" "CL05B104KB54PNC"
 			(at 302.26 53.34 90)
 			(hide yes)
@@
 			)
 		)
-		(property "JLCPCB Part #" "C105883"
+		(property "JLCPCB Part #" "C307331"
 			(at 302.26 53.34 90)
 			(hide yes)
@@
 			)
 		)
-		(property "MPN" "CC0402KRX7R8BB104"
+		(property "MPN" "CL05B104KB54PNC"
 			(at 273.05 217.17 90)
 			(hide yes)
@@
 			)
 		)
-		(property "JLCPCB Part #" "C105883"
+		(property "JLCPCB Part #" "C307331"
 			(at 273.05 217.17 90)
 			(hide yes)
@@
 		(body_style 1)
 		(exclude_from_sim no)
-		(in_bom yes)
+		(in_bom no)
 		(on_board yes)
 		(in_pos_files yes)
@@
 			)
 		)
-		(property "MPN" "RC0402FR-0710KL"
+		(property "MPN" "0402WGF1002TCE"
 			(at 97.79 193.04 90)
 			(hide yes)
@@
 			)
 		)
-		(property "JLCPCB Part #" "C60490"
+		(property "JLCPCB Part #" "C25744"
 			(at 97.79 193.04 90)
 			(hide yes)
@@
 			)
 		)
-		(property "MPN" "RC0402FR-0710KL"
+		(property "MPN" "0402WGF1002TCE"
 			(at 97.79 127 90)
 			(hide yes)
@@
 			)
 		)
-		(property "JLCPCB Part #" "C60490"
+		(property "JLCPCB Part #" "C25744"
 			(at 97.79 127 90)
 			(hide yes)
@@
 			)
 		)
-		(property "Voltage" "10V"
+		(property "Voltage" "50V"
 			(at 236.22 229.616 0)
 			(show_name no)
@@
 			)
 		)
-		(property "JLCPCB Part #" "C5137480"
+		(property "JLCPCB Part #" "C15195"
 			(at 241.3 227.33 0)
 			(hide yes)
@@
 			)
 		)
-		(property "MPN" "CC0402KRX7R8BB104"
+		(property "MPN" "CL05B104KB54PNC"
 			(at 285.75 217.17 90)
 			(hide yes)
@@
 			)
 		)
-		(property "JLCPCB Part #" "C105883"
+		(property "JLCPCB Part #" "C307331"
 			(at 285.75 217.17 90)
 			(hide yes)
@@
 			)
 		)
-		(property "MPN" "RT0402BRD078K2L"
+		(property "MPN" "0402WGF8201TCE"
 			(at 309.88 198.12 90)
 			(hide yes)
@@
 			)
 		)
-		(property "JLCPCB Part #" "C852943"
+		(property "JLCPCB Part #" "C25924"
 			(at 309.88 198.12 90)
 			(hide yes)
@@
 			)
 		)
-		(property "MPN" "CC0402KRX7R8BB104"
+		(property "MPN" "CL05B104KB54PNC"
 			(at 302.26 102.87 90)
 			(hide yes)
@@
 			)
 		)
-		(property "JLCPCB Part #" "C105883"
+		(property "JLCPCB Part #" "C307331"
 			(at 302.26 102.87 90)
 			(hide yes)
@@
 			)
 		)
-		(property "MPN" "RT0402BRD078K2L"
+		(property "MPN" "0402WGF8201TCE"
 			(at 297.18 210.82 0)
 			(hide yes)
@@
 			)
 		)
-		(property "JLCPCB Part #" "C852943"
+		(property "JLCPCB Part #" "C25924"
 			(at 297.18 210.82 0)
 			(hide yes)
@@
 			)
 		)
-		(property "MPN" "CC0402KRX7R8BB104"
+		(property "MPN" "CL05B104KB54PNC"
 			(at 119.38 172.72 0)
 			(hide yes)
@@
 			)
 		)
-		(property "JLCPCB Part #" "C105883"
+		(property "JLCPCB Part #" "C307331"
 			(at 119.38 172.72 0)
 			(hide yes)
@@
 			)
 		)
-		(property "MPN" "RC0402FR-0710KL"
+		(property "MPN" "0402WGF1002TCE"
 			(at 97.79 60.96 90)
 			(hide yes)
@@
 			)
 		)
-		(property "JLCPCB Part #" "C60490"
+		(property "JLCPCB Part #" "C25744"
 			(at 97.79 60.96 90)
 			(hide yes)
