File: Hardware/Digichiver.kicad_pcb (KiCad board)
At the start: 4 copper layers, 119 parts, among them J1 DM3AT-SF-PEJM5, J2 USB4105-GF-A, J3 61300211121, J4 61300211121, J5 SJ1-3535NG, SW1 PTS_647_SN50_SMTR2_LFS, SW2 PTS_647_SN50_SMTR2_LFS, SW3 PTS_647_SN50_SMTR2_LFS, U1 RP2354B, U10 TLV9004IPWR, U11 PAM8302AAD, U2 SN74LVC245A, U3 SN74LVC245A, U4 SN74LVC8T245, U5 SN74LVC8T245, U6 SN74LVC8T245, U7 TLV61046A, U8 TPSM84338, U9 PCM1809, X1 ICSockets-40P, X2 ABM8-272-T3

Commit message: layout complete
Parts:
- removed the C24 at (0.94, 0.48)
- removed the C25 at (0.94, 2.46)
- removed the C26 at (0.94, 4.42)
- added MNT1: MountingHole_2.7mm_M2.5, MountingHole:MountingHole_2.7mm_M2.5, F.Cu at (169.7, 63.5)
- added MNT2: MountingHole_2.7mm_M2.5, MountingHole:MountingHole_2.7mm_M2.5, F.Cu at (101.6, 63.5)
- added MNT3: MountingHole_2.7mm_M2.5, MountingHole:MountingHole_2.7mm_M2.5, F.Cu at (101.6, 141.5)
- added MNT4: MountingHole_2.7mm_M2.5, MountingHole:MountingHole_2.7mm_M2.5, F.Cu at (186.4, 141.5)
- C1, C10, C2, C3, C30, C32, C33, C34, C35, C39, C4, C40, C41, C42, C47, C48, C5, C54, C55, C6, C7, C8, C9, R10, R19, R20, R21, R22, R23, R34, R35, R36: moved to B.Cu
- U2, U3, U4, U5, U6: moved to F.Cu
- moved R5 150.2 mm to (107.4, 133.1), turned to 180 degrees
- moved R4 138.3 mm to (99.3, 108.7), turned to 180 degrees
- moved R11 134.1 mm to (127.8, 71.1), turned to 90 degrees
- moved X2 129.7 mm to (130.2, 87.4), turned to -90 degrees
- moved R6 128.2 mm to (130.6, 84.6)
- moved R3 124.1 mm to (101.9, 72.1), turned to 90 degrees
- moved LS1 123.1 mm to (157.5, 130.8)
- moved C6 122.8 mm to (98.0, 107.2), turned to 90 degrees
- moved C8 122.0 mm to (106.2, 131.6), turned to 90 degrees
- moved C9 121.9 mm to (107.7, 122.4)
- moved C7 119.0 mm to (99.6, 98.3)
- moved R1 113.9 mm to (140.5, 119.1), turned to -90 degrees
- moved C5 113.6 mm to (103.4, 70.9)
- moved SW1 112.5 mm to (142.3, 62.2)
- moved U9 110.1 mm to (150.6, 80.4), turned to -90 degrees
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- renumbered X1 to XC1
Connections:
- U1 pad 20: /~{ROMEN} -> /ROM_ADDR0
- U1 pad 21: /INTR -> /ROM_ADDR1
- U1 pad 22: /ROM_ADDR0 -> /ROM_ADDR2
- U1 pad 23: /ROM_ADDR1 -> /ROM_ADDR3
- U1 pad 25: /ROM_ADDR2 -> /ROM_ADDR4
- U1 pad 26: /ROM_ADDR3 -> /ROM_ADDR5
- U1 pad 27: /ROM_ADDR4 -> /ROM_ADDR6
- U1 pad 28: /ROM_ADDR5 -> /ROM_ADDR7
- U1 pad 36: /ROM_ADDR6 -> /ROM_ADDR8
- U1 pad 37: /ROM_ADDR7 -> /ROM_ADDR9
- U1 pad 38: /ROM_ADDR8 -> /ROM_ADDR10
- U1 pad 39: /ROM_ADDR9 -> /ROM_ADDR11
- U1 pad 40: /ROM_ADDR10 -> /ROM_ADDR12
- U1 pad 42: /ROM_ADDR11 -> /ROM_ADDR13
- U1 pad 43: /ROM_ADDR12 -> /~{ROMEN}
- U1 pad 44: /ROM_ADDR13 -> /INTR
- U1 pad 45: /SDATA -> /FSYNC
- U1 pad 46: /FSYNC -> /BCLK
- U1 pad 47: /BCLK -> /SDATA
- U9 pad 3: Net-(U9-IN2M) -> Net-(U9-IN2P)
- U9 pad 4: (no net) -> Net-(U9-IN2M)
Routing:
- net GND: track 0.97 -> 158.3 mm, vias 3 -> 60
- net +5V: track 0.00 -> 98.2 mm, vias 0 -> 11
- net /Control/LED_GR: track 0.00 -> 81.7 mm, vias 0 -> 2
- net /Control/LED_RED: track 0.00 -> 80.8 mm, vias 0 -> 2
- net /Control/BUTTON: track 0.00 -> 79.4 mm, vias 0 -> 2
- net /Digitalker/FILTERED_SPEECH: track 0.00 -> 64.4 mm, vias 0 -> 1
- net /RDATA0: track 0.00 -> 63.0 mm
- net /RDATA1: track 0.00 -> 62.4 mm
- net /RDATA2: track 0.00 -> 61.8 mm
- net /RDATA3: track 0.00 -> 61.2 mm
- net /RDATA4: track 0.00 -> 60.5 mm
- net /RDATA5: track 0.00 -> 59.8 mm
- net /RDATA6: track 0.00 -> 59.2 mm
- net /RDATA7: track 0.00 -> 58.6 mm
- net /Control/SD_DET: track 0.00 -> 57.4 mm, vias 0 -> 2
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- added copper zone on In2.Cu, net +3.3V
- added copper zone on In2.Cu, net +5V
- added copper zone on F.Cu, net /Power/+3V3_RAW
- added copper zone on In1.Cu, net GND
Other:
- board outline added: 95 x 88.1 mm
- board text added: "+9V EN"
- board text added: "3.3V EN"
- board text added: "BOOT SEL"
- board text added: "RST"

Commit message: ac couple speaker amp input
Parts:
- added C56: 1uF, Capacitor_SMD:C_0402_1005Metric, F.Cu at (160.0, 102.2)
Connections:
- U11 pad 4: GND -> Net-(U11-IN-)
Routing:
- net Net-(U11-IN-): track 0.00 -> 1.91 mm

Commit message: add title silk
Other:
- board text added: "B0"
- board text added: "Digichiver Rev. 0"
Changed lines of the file:
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@@
 		)
 	)
+	(gr_text "Digichiver\nRev. 0"
+		(at 170.688 143.764 0)
+		(layer "F.SilkS")
+		(effects
+			(font
+				(size 1.5 1.5)
+				(thickness 0.3)
+				(bold yes)
+			)
+			(justify left bottom)
+		)
+	)
+	(gr_text "B0"
+		(at 175.514 126.492 0)
+		(layer "F.SilkS")
+		(effects
+			(font
+				(size 1.5 1.5)
+				(thickness 0.3)
+				(bold yes)
+			)
+			(justify left bottom)
+		)
+	)
 	(gr_text "+9V\nEN"
 		(at 118.618 72.898 0)
@@
 	)
 	(segment
+		(start 160.013 102.685)
+		(end 159.997 102.669)
+		(width 0.2)
+		(layer "F.Cu")
+		(net "Net-(U11-IN-)")
+	)
+	(segment
+		(start 160.013 104.5675)
+		(end 160.013 102.685)
+		(width 0.2)
+		(layer "F.Cu")
+		(net "Net-(U11-IN-)")
+	)
+	(segment
 		(start 129.75 72.39)
 		(end 128.99 71.63)
@@
 		(net "Net-(C55-Pad1)")
 	)
-	(segment
-		(start 160.013 102.685)
-		(end 159.997 102.669)
-		(width 0.2)
-		(layer "F.Cu")
-		(net "Net-(U11-IN-)")
-	)
-	(segment
-		(start 160.013 104.5675)
-		(end 160.013 102.685)
-		(width 0.2)
-		(layer "F.Cu")
-		(net "Net-(U11-IN-)")
-	)
 	(zone

Commit message: swap D2 to amber, silk text
Parts:
- D2: value 150060RS75000 -> 150060AS75000
Other:
- board text added: "ACTIVITY"
- board text added: "READY"
Changed lines of the file:
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@@
 			)
 		)
-		(property "Value" "150060RS75000"
+		(property "Value" "150060AS75000"
 			(at 0 1.43 90)
 			(layer "F.Fab")
@@
 		)
 	)
+	(gr_text "ACTIVITY"
+		(at 183.896 124.968 90)
+		(layer "F.SilkS")
+		(effects
+			(font
+				(size 1.5 1.5)
+				(thickness 0.3)
+				(bold yes)
+			)
+			(justify right bottom)
+		)
+	)
+	(gr_text "READY"
+		(at 188.976 124.968 90)
+		(layer "F.SilkS")
+		(effects
+			(font
+				(size 1.5 1.5)
+				(thickness 0.3)
+				(bold yes)
+			)
+			(justify right bottom)
+		)
+	)
