File: Hardware/Digichiver.kicad_pcb (KiCad board)
At the start: 4 copper layers, 95 x 88.1 mm, 121 parts, among them J1 DM3AT-SF-PEJM5, J2 USB4105-GF-A, J3 61300211121, J4 61300211121, J5 SJ1-3535NG, SW1 PTS_647_SN50_SMTR2_LFS, SW2 PTS_647_SN50_SMTR2_LFS, SW3 PTS_647_SN50_SMTR2_LFS, U1 RP2354B, U10 TLV9004IPWR, U11 PAM8302AAD, U2 SN74LVC245A, U3 SN74LVC245A, U4 SN74LVC8T245, U5 SN74LVC8T245, U6 SN74LVC8T245, U7 TLV61046A, U8 TPSM84338, U9 PCM1809, X2 ABM8-272-T3

Commit message: generate Rev1 outputs
Parts:
- U11: value PAM8302AAD -> PAM8302AASCR
Changed lines of the file:
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@@
 		(tags "Integrated Circuit")
 		(property "Reference" "U9"
-			(at 0 0 270)
+			(at 0 0 90)
 			(layer "F.SilkS")
 			(hide yes)
@@
 		)
 		(property "Value" "PCM1809"
-			(at 0 0 270)
+			(at 0 0 90)
 			(layer "F.SilkS")
 			(hide yes)
@@
 		)
 		(property "Datasheet" "https://www.ti.com/lit/ds/symlink/pcm1809.pdf?ts=1723810813788"
-			(at 0 0 270)
+			(at 0 0 90)
 			(layer "F.Fab")
 			(hide yes)
@@
 		)
 		(property "Description" ""
-			(at 0 0 270)
+			(at 0 0 90)
 			(layer "F.Fab")
 			(hide yes)
@@
 		(sheetname "/Audio/")
 		(sheetfile "Audio.kicad_sch")
-		(units
-			(unit
-				(name "A")
-				(pins "9" "16" "1" "2" "3" "4" "11" "12" "13" "19" "17" "14" "6" "7"
-					"8" "18" "5" "10" "15" "20" "21"
-				)
-			)
-		)
 		(attr smd)
 		(duplicate_pad_numbers_are_jumpers no)
@@
 			(layer "F.Fab")
 		)
+		(fp_text user "U9"
+			(at -0.044 2.667 270)
+			(layer "F.SilkS")
+			(effects
+				(font
+					(size 1 1)
+					(thickness 0.15)
+				)
+			)
+		)
 		(fp_text user "${REFERENCE}"
-			(at 0 0 270)
+			(at 0 0 90)
 			(layer "F.Fab")
 			(effects
@@
 			)
 		)
-		(property "Value" "PAM8302AAD"
+		(property "Value" "PAM8302AASCR"
 			(at 0 2.45 90)
 			(layer "F.Fab")
@@
 			)
 		)
-		(property "MPN" "PAM8302AADCR "
+		(property "MPN" "PAM8302AASCR"
 			(at 0 0 270)
 			(unlocked yes)
@@
 			)
 		)
-		(property "JLCPCB Part #" "C112137"
+		(property "JLCPCB Part #" "C113367"
 			(at 0 0 270)
 			(unlocked yes)
@@
 	)
 	(segment
+		(start 136.712 75.632)
+		(end 134.49 75.632)
+		(width 0.2)
+		(layer "F.Cu")
+		(net "/Control/LED_OR")
+	)
+	(segment
+		(start 183.134 119.124)
+		(end 183.134 118.364)
+		(width 0.1778)
+		(layer "F.Cu")
+		(net "/Control/LED_OR")
+	)
+	(segment
+		(start 137.414 74.93)
+		(end 136.712 75.632)
+		(width 0.2)
+		(layer "F.Cu")
+		(net "/Control/LED_OR")
+	)
+	(via
+		(at 137.414 74.93)
+		(size 0.45)
+		(drill 0.3)
+		(layers "F.Cu" "B.Cu")
+		(net "/Control/LED_OR")
+	)
+	(via
+		(at 183.134 118.364)
+		(size 0.45)
+		(drill 0.3)
+		(layers "F.Cu" "B.Cu")
+		(net "/Control/LED_OR")
+	)
+	(segment
+		(start 169.418 110.49)
+		(end 169.418 88.138)
+		(width 0.1778)
+		(layer "B.Cu")
+		(net "/Control/LED_OR")
+	)
+	(segment
+		(start 173.228 114.3)
+		(end 169.418 110.49)
+		(width 0.1778)
+		(layer "B.Cu")
+		(net "/Control/LED_OR")
+	)
+	(segment
+		(start 138.033765 74.93)
+		(end 137.414 74.93)
+		(width 0.1778)
+		(layer "B.Cu")
+		(net "/Control/LED_OR")
+	)
+	(segment
+		(start 183.134 118.364)
+		(end 179.07 114.3)
+		(width 0.1778)
+		(layer "B.Cu")
+		(net "/Control/LED_OR")
+	)
+	(segment
+		(start 150.114 78.232)
+		(end 141.335765 78.232)
+		(width 0.1778)
+		(layer "B.Cu")
+		(net "/Control/LED_OR")
+	)
+	(segment
+		(start 169.418 88.138)
+		(end 164.846 83.566)
+		(width 0.1778)
+		(layer "B.Cu")
+		(net "/Control/LED_OR")
+	)
+	(segment
+		(start 179.07 114.3)
+		(end 173.228 114.3)
+		(width 0.1778)
+		(layer "B.Cu")
+		(net "/Control/LED_OR")
+	)
+	(segment
+		(start 164.846 83.566)
+		(end 155.448 83.566)
+		(width 0.1778)
+		(layer "B.Cu")
+		(net "/Control/LED_OR")
+	)
+	(segment
+		(start 155.448 83.566)
+		(end 150.114 78.232)
+		(width 0.1778)
+		(layer "B.Cu")
+		(net "/Control/LED_OR")
+	)
+	(segment
+		(start 141.335765 78.232)
+		(end 138.033765 74.93)
+		(width 0.1778)
+		(layer "B.Cu")
+		(net "/Control/LED_OR")
+	)
+	(segment
 		(start 130.79 65.656)
 		(end 130.79 64.536)
@@
 		(net "Net-(C55-Pad1)")
 	)
-	(segment
-		(start 136.712 75.632)
-		(end 134.49 75.632)
-		(width 0.2)
-		(layer "F.Cu")
-		(net "/Control/LED_OR")
-	)
-	(segment
-		(start 183.134 119.124)
-		(end 183.134 118.364)
-		(width 0.1778)
-		(layer "F.Cu")
-		(net "/Control/LED_OR")
-	)
-	(segment
-		(start 137.414 74.93)
-		(end 136.712 75.632)
-		(width 0.2)
-		(layer "F.Cu")
-		(net "/Control/LED_OR")
-	)
-	(via
-		(at 137.414 74.93)
-		(size 0.45)
-		(drill 0.3)
-		(layers "F.Cu" "B.Cu")
-		(net "/Control/LED_OR")
-	)
-	(via
-		(at 183.134 118.364)
-		(size 0.45)
-		(drill 0.3)
-		(layers "F.Cu" "B.Cu")
-		(net "/Control/LED_OR")
-	)
-	(segment
-		(start 169.418 110.49)
-		(end 169.418 88.138)
-		(width 0.1778)
-		(layer "B.Cu")
-		(net "/Control/LED_OR")
-	)
-	(segment
-		(start 173.228 114.3)
-		(end 169.418 110.49)
-		(width 0.1778)
-		(layer "B.Cu")
-		(net "/Control/LED_OR")
-	)
-	(segment
-		(start 138.033765 74.93)
-		(end 137.414 74.93)
-		(width 0.1778)
-		(layer "B.Cu")
-		(net "/Control/LED_OR")
-	)
-	(segment
-		(start 183.134 118.364)
-		(end 179.07 114.3)
-		(width 0.1778)
-		(layer "B.Cu")
-		(net "/Control/LED_OR")
-	)
-	(segment
-		(start 150.114 78.232)
-		(end 141.335765 78.232)
-		(width 0.1778)
-		(layer "B.Cu")
-		(net "/Control/LED_OR")
-	)
-	(segment
-		(start 169.418 88.138)
-		(end 164.846 83.566)
-		(width 0.1778)
-		(layer "B.Cu")
-		(net "/Control/LED_OR")
-	)
-	(segment
-		(start 179.07 114.3)
-		(end 173.228 114.3)
-		(width 0.1778)
-		(layer "B.Cu")
-		(net "/Control/LED_OR")
-	)
-	(segment
-		(start 164.846 83.566)
-		(end 155.448 83.566)
-		(width 0.1778)
-		(layer "B.Cu")
-		(net "/Control/LED_OR")
-	)
-	(segment
-		(start 155.448 83.566)
-		(end 150.114 78.232)
-		(width 0.1778)
-		(layer "B.Cu")
-		(net "/Control/LED_OR")
-	)
-	(segment
-		(start 141.335765 78.232)
-		(end 138.033765 74.93)
-		(width 0.1778)
-		(layer "B.Cu")
-		(net "/Control/LED_OR")
-	)
 	(zone
