File: Hardware/Digichiver.kicad_pcb (KiCad board)
At the start: 4 copper layers, 95 x 88.1 mm, 121 parts, among them J1 DM3AT-SF-PEJM5, J2 USB4105-GF-A, J3 61300211121, J4 61300211121, J5 SJ1-3535NG, SW1 PTS_647_SN50_SMTR2_LFS, SW2 PTS_647_SN50_SMTR2_LFS, SW3 PTS_647_SN50_SMTR2_LFS, U1 RP2354B, U10 TLV9004IPWR, U11 PAM8302AASCR, U2 SN74LVC245A, U3 SN74LVC245A, U4 SN74LVC8T245, U5 SN74LVC8T245, U6 SN74LVC8T245, U7 TLV61046A, U8 TPSM84338, U9 PCM1809, X2 ABM8-272-T3

Commit message: rev2
move all components to top side and update BOM to use basic JLCPCB components when possible
Parts:
- C1, C10, C15, C16, C17, C18, C19, C2, C20, C21, C22, C23, C24, C25, C26, C3, C30, C32, C33, C35, C4, C40, C41, C42, C47, C5, C54, C55, C6, C7, C8, C9, R10, R19, R20, R21, R22, R23, R34, R35, R36: moved to F.Cu
- C31, C37, C38: footprint Capacitor_SMD:C_0402_1005Metric -> Capacitor_SMD:C_0603_1608Metric
- C34: footprint Capacitor_SMD:C_0402_1005Metric -> Capacitor_SMD:C_0805_2012Metric; moved to F.Cu
- C39, C48: footprint Capacitor_SMD:C_0402_1005Metric -> Capacitor_SMD:C_0603_1608Metric; moved to F.Cu
- D1: value 150060VS75000 -> KT-0805G; footprint LED_SMD:LED_0603_1608Metric -> LED_SMD:LED_0805_2012Metric
- D2: value 150060AS75000 -> KT-0805Y; footprint LED_SMD:LED_0603_1608Metric -> LED_SMD:LED_0805_2012Metric
- R13: value 133 -> 1k
- R33: value 133 -> 150
- R8, R9: footprint Resistor_SMD:R_0402_1005Metric -> Resistor_SMD:R_0603_1608Metric
- SW1, SW2, SW3: value PTS_647_SN50_SMTR2_LFS -> TS-1088-AR02016; footprint Button_Switch_SMD:SW_SPST_PTS647_Sx50 -> Button_Switch_SMD:SW_SPST_TS-1088-xR020
- moved C41 15.6 mm to (157.1, 99.2), turned to -90 degrees
- moved R23 15.1 mm to (157.6, 97.5)
- moved C42 14.6 mm to (159.8, 98.7)
- moved R21 14.6 mm to (159.8, 101.2)
- moved R22 14.6 mm to (159.8, 99.9)
- moved R35 10.9 mm to (173.0, 69.8)
- moved R34 7.89 mm to (170.9, 69.3)
- moved R20 7.55 mm to (135.5, 61.3), turned to -90 degrees
- moved R36 7.38 mm to (169.4, 70.4)
- moved C2 7.26 mm to (140.5, 109.2), turned to 180 degrees
- moved C1 7.16 mm to (147.7, 98.8), turned to 180 degrees
- moved C55 6.87 mm to (167.4, 69.8)
- moved C47 5.45 mm to (156.1, 87.6), turned to 0 degrees
- moved C30 5.34 mm to (171.4, 85.5), turned to 180 degrees
- moved R19 5.21 mm to (135.5, 63.4), turned to 90 degrees
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Connections:
- net /Control/LED_OR renamed /Control/LED_YEL
- SW1 pad 2: GND -> Net-(R11-Pad2)
- SW2 pad 2: Net-(R10-Pad2) -> Net-(U1-RUN)
- SW3 pad 2: /Control/BUTTON -> +3.3V
Routing:
- net GND: track 159.1 -> 143.1 mm, vias 61 -> 71
- net /Digitalker/V_BIAS: track 19.8 -> 4.85 mm, vias 1 -> 0
- net Net-(XC1-SPEECH_OUT): track 5.89 -> 19.8 mm, vias 0 -> 1
- net Net-(J5-PadT): track 3.03 -> 14.2 mm
- net Net-(U10A-+): track 19.1 -> 9.81 mm, vias 1 -> 2
- net Net-(U1-RUN): track 50.7 -> 42.4 mm
- net Net-(J5-PadR): track 2.70 -> 10.8 mm
- net Net-(J2-CC2): track 2.17 -> 9.65 mm, vias 1 -> 0
- net +3.3V: track 66.3 -> 59.0 mm, vias 32 -> 35
- net /Digitalker/FILTERED_SPEECH: track 64.4 -> 58.2 mm, vias 1 -> 2
- net /Control/XOUT: track 1.53 -> 7.36 mm
- net /Control/XR: track 6.96 -> 2.75 mm
- net Net-(J2-CC1): track 2.17 -> 6.23 mm, vias 1 -> 0
- net Net-(C55-Pad1): track 8.67 -> 4.60 mm
- net /Power/+3V3_RAW: track 5.93 -> 9.92 mm, vias 1 -> 0
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- removed copper zone on F.Cu, net /Power/+3V3_RAW
Other:
- board size 95 x 88.1 mm -> 96.9 x 88.1 mm
- board text added: "Digichiver Rev. 2"
- board text removed: "Digichiver Rev. 1"
