File: Hardware/Audio.kicad_sch (KiCad schematic)
At the start: 21 parts, among them J5 SJ1-3535NG, U11 PAM8302AAD, U9 PCM1809

Commit message: comment clarification
Other:
- note added: "OUT TO EXTERRNAL SPEAKER AMPLIFIER"
- note removed: "OUT TO EXTERRNAL SPEAKER"
Changed lines of the file:
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@@
 		(company "J. Thweatt")
 	)
-	(text "OUT TO EXTERRNAL SPEAKER"
+	(text "OUT TO EXTERRNAL SPEAKER AMPLIFIER"
 		(exclude_from_sim no)
-		(at 271.526 137.668 0)
+		(at 277.622 136.144 0)
 		(effects
 			(font
