File: Hardware/Audio.kicad_sch (KiCad schematic)
At the start: 21 parts, among them J5 SJ1-3535NG, U11 PAM8302AAD, U9 PCM1809

Commit message: update PCM1809 footprint
Parts:
- U9: footprint Package_DFN_QFN:WQFN-20-1EP_3x3mm_P0.4mm_EP1.7x1.7mm -> Digichiver:PCM1820IRTER
Changed lines of the file:
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@@
 			)
 		)
-		(property "Footprint" "Package_DFN_QFN:WQFN-20-1EP_3x3mm_P0.4mm_EP1.7x1.7mm"
+		(property "Footprint" "Digichiver:PCM1820IRTER"
 			(at 209.55 71.12 0)
 			(hide yes)

Commit message: generate Rev1 outputs
Parts:
- U11: value PAM8302AAD -> PAM8302AASCR; JLCPCB Part # C112137 -> C113367; MPN PAM8302AADCR -> PAM8302AASCR
Changed lines of the file:
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@@
 			)
 		)
-		(property "Value" "PAM8302AAD"
+		(property "Value" "PAM8302AASCR"
 			(at 211.6933 168.91 0)
 			(show_name no)
@@
 			)
 		)
-		(property "MPN" "PAM8302AADCR "
+		(property "MPN" "PAM8302AASCR"
 			(at 209.55 179.07 0)
 			(hide yes)
@@
 			)
 		)
-		(property "JLCPCB Part #" "C112137"
+		(property "JLCPCB Part #" "C113367"
 			(at 209.55 179.07 0)
 			(hide yes)

Commit message: rev2
move all components to top side and update BOM to use basic JLCPCB components when possible
Parts:
- C37, C38, C39: footprint Capacitor_SMD:C_0402_1005Metric -> Capacitor_SMD:C_0603_1608Metric; JLCPCB Part # C315248 -> C96446; MPN CL05A106MP5NUNC -> CL10A106MA8NRNC; Voltage 10V -> 25V
- C54: JLCPCB Part # C105883 -> C307331; MPN CC0402KRX7R8BB104 -> CL05B104KB54PNC
- R34, R35: JLCPCB Part # C106232 -> C25076; MPN RC0402FR-07100RL -> 0402WGF1000TCE
- R36: JLCPCB Part # C60491 -> C25741; MPN RC0402FR-07100KL -> 0402WGF1003TCE
Changed lines of the file:
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@@
 	(title_block
 		(title "Digichiver")
-		(date "2026-07-24")
-		(rev "1")
+		(date "2026-09-01")
+		(rev "2")
 		(company "J. Thweatt")
 	)
@@
 			)
 		)
-		(property "MPN" "CC0402KRX7R8BB104"
+		(property "MPN" "CL05B104KB54PNC"
 			(at 204.47 161.29 0)
 			(hide yes)
@@
 			)
 		)
-		(property "JLCPCB Part #" "C105883"
+		(property "JLCPCB Part #" "C307331"
 			(at 204.47 161.29 0)
 			(hide yes)
@@
 			)
 		)
-		(property "Footprint" "Capacitor_SMD:C_0402_1005Metric"
+		(property "Footprint" "Capacitor_SMD:C_0603_1608Metric"
 			(at 233.3752 73.66 0)
 			(hide yes)
@@
 			)
 		)
-		(property "Voltage" "10V"
+		(property "Voltage" "25V"
 			(at 237.49 72.136 0)
 			(show_name no)
@@
 			)
 		)
-		(property "MPN" "CL05A106MP5NUNC"
+		(property "MPN" "CL10A106MA8NRNC"
 			(at 232.41 69.85 0)
 			(hide yes)
@@
 			)
 		)
-		(property "JLCPCB Part #" "C315248"
+		(property "JLCPCB Part #" "C96446"
 			(at 232.41 69.85 0)
 			(hide yes)
@@
 			)
 		)
-		(property "MPN" "RC0402FR-07100RL"
+		(property "MPN" "0402WGF1000TCE"
 			(at 234.95 129.54 90)
 			(hide yes)
@@
 			)
 		)
-		(property "JLCPCB Part #" "C106232"
+		(property "JLCPCB Part #" "C25076"
 			(at 234.95 129.54 90)
 			(hide yes)
@@
 			)
 		)
-		(property "MPN" "RC0402FR-07100KL"
+		(property "MPN" "0402WGF1003TCE"
 			(at 223.52 140.97 0)
 			(hide yes)
@@
 			)
 		)
-		(property "JLCPCB Part #" "C60491"
+		(property "JLCPCB Part #" "C25741"
 			(at 223.52 140.97 0)
 			(hide yes)
@@
 			)
 		)
-		(property "MPN" "RC0402FR-07100RL"
+		(property "MPN" "0402WGF1000TCE"
 			(at 234.95 134.62 90)
 			(hide yes)
@@
 			)
 		)
-		(property "JLCPCB Part #" "C106232"
+		(property "JLCPCB Part #" "C25076"
 			(at 234.95 134.62 90)
 			(hide yes)
@@
 			)
 		)
-		(property "Footprint" "Capacitor_SMD:C_0402_1005Metric"
+		(property "Footprint" "Capacitor_SMD:C_0603_1608Metric"
 			(at 187.6552 73.66 0)
 			(hide yes)
@@
 			)
 		)
-		(property "Voltage" "10V"
+		(property "Voltage" "25V"
 			(at 181.102 72.136 0)
 			(show_name no)
@@
 			)
 		)
-		(property "MPN" "CL05A106MP5NUNC"
+		(property "MPN" "CL10A106MA8NRNC"
 			(at 186.69 69.85 0)
 			(hide yes)
@@
 			)
 		)
-		(property "JLCPCB Part #" "C315248"
+		(property "JLCPCB Part #" "C96446"
 			(at 186.69 69.85 0)
 			(hide yes)
@@
 			)
 		)
-		(property "Footprint" "Capacitor_SMD:C_0402_1005Metric"
+		(property "Footprint" "Capacitor_SMD:C_0603_1608Metric"
 			(at 246.0752 73.66 0)
 			(hide yes)
@@
 			)
 		)
-		(property "Voltage" "10V"
+		(property "Voltage" "25V"
 			(at 250.19 72.136 0)
 			(show_name no)
@@
 			)
 		)
-		(property "MPN" "CL05A106MP5NUNC"
+		(property "MPN" "CL10A106MA8NRNC"
 			(at 245.11 69.85 0)
 			(hide yes)
@@
 			)
 		)
-		(property "JLCPCB Part #" "C315248"
+		(property "JLCPCB Part #" "C96446"
 			(at 245.11 69.85 0)
 			(hide yes)
