File: Hardware/Control.kicad_sch (KiCad schematic)
At the start: 43 parts, among them J1 DM3AT-SF-PEJM5, SW1 PTS_647_SN50_SMTR2_LFS, SW2 PTS_647_SN50_SMTR2_LFS, SW3 PTS_647_SN50_SMTR2_LFS, U1 RP2354B, X2 ABM8-272-T3

Commit message: update PCM1809 footprint
Connections:
- net BCLK: now also U1.45 (GPIO36); no longer U1.46 (GPIO37)
- net FSYNC: now also U1.46 (GPIO37); no longer U1.45 (GPIO36)
Changed lines of the file:
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@@
-		)
-	)
-	(label "BCLK"
-		(at 246.38 179.07 0)
-		(effects
-			(font
-				(size 1.27 1.27)
-			)
-			(justify left bottom)
 		)
 	)
@@
 		)
 	)
+	(label "FSYNC"
+		(at 246.38 179.07 0)
+		(effects
+			(font
+				(size 1.27 1.27)
+			)
+			(justify left bottom)
+		)
+	)
 	(label "~{DIGITALKER_CS}"
 		(at 246.38 87.63 0)
@@
 		)
 	)
+	(label "BCLK"
+		(at 246.38 176.53 0)
+		(effects
+			(font
+				(size 1.27 1.27)
+			)
+			(justify left bottom)
+		)
+	)
 	(label "SW1"
 		(at 246.38 95.25 0)
@@
 	(label "ROM_ADDR10"
 		(at 246.38 161.29 0)
-		(effects
-			(font
-				(size 1.27 1.27)
-			)
-			(justify left bottom)
-		)
-	)
-	(label "FSYNC"
-		(at 246.38 176.53 0)
 		(effects
 			(font
@@
 		)
 	)
+	(hierarchical_label "FSYNC"
+		(shape output)
+		(at 259.08 179.07 0)
+		(effects
+			(font
+				(size 1.27 1.27)
+			)
+			(justify left)
+		)
+	)
+	(hierarchical_label "BCLK"
+		(shape output)
+		(at 259.08 176.53 0)
+		(effects
+			(font
+				(size 1.27 1.27)
+			)
+			(justify left)
+		)
+	)
 	(hierarchical_label "DIGITALKER_CLK_4MHZ"
 		(shape output)
@@
 		)
 	)
-	(hierarchical_label "FSYNC"
-		(shape output)
-		(at 259.08 176.53 0)
-		(effects
-			(font
-				(size 1.27 1.27)
-			)
-			(justify left)
-		)
-	)
 	(hierarchical_label "~{ROMEN}"
 		(shape input)
@@
 		(effects
 			(font
-				(size 1.27 1.27)
-			)
-			(justify left)
-		)
-	)
-	(hierarchical_label "BCLK"
-		(shape output)
-		(at 259.08 179.07 0)
-		(effects
-			(font

Commit message: update orange LED net name
Parts:
- D2: Color AMBER -> ORANGE
Connections:
- net LED_RED renamed LED_OR
Changed lines of the file:
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@@
 		)
 	)
-	(label "LED_RED"
+	(label "LED_OR"
 		(at 121.92 157.48 0)
 		(effects
@@
 		)
 	)
-	(label "LED_RED"
+	(label "LED_OR"
 		(at 177.8 168.91 0)
 		(effects
@@
 			)
 		)
-		(property "Color" "AMBER"
+		(property "Color" "ORANGE"
 			(at 104.648 164.846 0)
 			(show_name no)

Commit message: rev2
move all components to top side and update BOM to use basic JLCPCB components when possible
Parts:
- C10, C11: JLCPCB Part # C106997 -> C1548; MPN CC0402JRNPO9BN150 -> 0402CG150J500NT; Voltage 10V -> 50V
- C12, C13, C14, C15: JLCPCB Part # C318563 -> C23733; MPN CL05A475MO5NUNC -> CL05A475MP5NRNC; Voltage 25V -> 10V
- C16, C17, C18, C19, C20, C21, C22, C23, C24, C25, C26, C29, C30: JLCPCB Part # C105883 -> C307331; MPN CC0402KRX7R8BB104 -> CL05B104KB54PNC
- C48: footprint Capacitor_SMD:C_0402_1005Metric -> Capacitor_SMD:C_0603_1608Metric; JLCPCB Part # C315248 -> C96446; MPN CL05A106MP5NUNC -> CL10A106MA8NRNC; Voltage 10V -> 25V
- D1: value 150060VS75000 -> KT-0805G; footprint LED_SMD:LED_0603_1608Metric -> LED_SMD:LED_0805_2012Metric; JLCPCB Part # C6848499 -> C2297; MPN 150060VS75000 -> KT-0805G
- D2: value 150060AS75000 -> KT-0805Y; footprint LED_SMD:LED_0603_1608Metric -> LED_SMD:LED_0805_2012Metric; Color ORANGE -> YELLOW; JLCPCB Part # C6976659 -> C2296; MPN 150060AS75000 -> KT-0805Y
- R10, R11, R6, R7: JLCPCB Part # C105637 -> C11702; MPN RC0402JR-071KL -> 0402WGF1001TCE
- R12, R28, R29, R30, R31, R32: JLCPCB Part # C60490 -> C25744; MPN RC0402FR-0710KL -> 0402WGF1002TCE
- R13: value 133 -> 1k; JLCPCB Part # C327373 -> C11702; MPN RC0402FR-07133RL -> 0402WGF1001TCE
- R33: value 133 -> 150; JLCPCB Part # C327373 -> C25082; MPN RC0402FR-07133RL -> 0402WGF1500TCE
- R8, R9: footprint Resistor_SMD:R_0402_1005Metric -> Resistor_SMD:R_0603_1608Metric; JLCPCB Part # C138021 -> C25190; MPN RC0402FR-0727RL -> 0603WAF270JT5E
- SW1, SW2, SW3: value PTS_647_SN50_SMTR2_LFS -> TS-1088-AR02016; footprint Button_Switch_SMD:SW_SPST_PTS647_Sx50 -> Button_Switch_SMD:SW_SPST_TS-1088-xR020; JLCPCB Part # C2799414 -> C720477; MPN PTS_647_SN50_SMTR2_LFS -> TS-1088-AR02016
Connections:
- net +3.3V: now also SW3.2; no longer SW3.3, SW3.4
- net BUTTON: no longer SW3.2
- net GND: no longer SW1.2
- net at R10.2, SW2.1: no longer SW2.2
- net LED_OR renamed LED_YEL
- new net: R11.2, SW1.2
- new net: SW2.2, U1.35 (RUN)
