File: Hardware/Power.kicad_sch (KiCad schematic)
At the start: 15 parts, among them J3 61300211121, J4 61300211121, U7 TLV61046A, U8 TPSM84338

Commit message: fix power jumper footprints
Parts:
- J3, J4: footprint Connector_PinHeader_1.00mm:PinHeader_1x02_P1.00mm_Vertical -> Connector_PinHeader_2.54mm:PinHeader_1x02_P2.54mm_Vertical
Changed lines of the file:
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@@
 			)
 		)
-		(property "Footprint" "Connector_PinHeader_1.00mm:PinHeader_1x02_P1.00mm_Vertical"
+		(property "Footprint" "Connector_PinHeader_2.54mm:PinHeader_1x02_P2.54mm_Vertical"
 			(at 247.65 163.83 0)
 			(hide yes)
@@
 			)
 		)
-		(property "Footprint" "Connector_PinHeader_1.00mm:PinHeader_1x02_P1.00mm_Vertical"
+		(property "Footprint" "Connector_PinHeader_2.54mm:PinHeader_1x02_P2.54mm_Vertical"
 			(at 261.62 102.87 0)
 			(hide yes)

Commit message: rev2
move all components to top side and update BOM to use basic JLCPCB components when possible
Parts:
- C31: footprint Capacitor_SMD:C_0402_1005Metric -> Capacitor_SMD:C_0603_1608Metric; JLCPCB Part # C315248 -> C96446; MPN CL05A106MP5NUNC -> CL10A106MA8NRNC; Voltage 10V -> 25V
- C32, C35: Voltage 10V -> 6.3V
- C34: footprint Capacitor_SMD:C_0402_1005Metric -> Capacitor_SMD:C_0805_2012Metric; JLCPCB Part # C318563 -> C1779; MPN CL05A475MO5NUNC -> CL21A475KAQNNNE
- J3, J4: now left out of the parts list
- R15: JLCPCB Part # C138044 -> C25762; MPN RC0402FR-0718KL -> 0402WGF1802TCE
- R18: JLCPCB Part # C60490 -> C25744; MPN RC0402FR-0710KL -> 0402WGF1002TCE
Changed lines of the file:
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@@
 	(title_block
 		(title "Digichiver")
-		(date "2026-07-24")
-		(rev "1")
+		(date "2026-09-01")
+		(rev "2")
 		(company "J. Thweatt")
 	)
@@
 			)
 		)
-		(property "Footprint" "Capacitor_SMD:C_0402_1005Metric"
+		(property "Footprint" "Capacitor_SMD:C_0805_2012Metric"
 			(at 234.6452 167.64 0)
 			(hide yes)
@@
 			)
 		)
-		(property "MPN" "CL05A475MO5NUNC"
+		(property "MPN" "CL21A475KAQNNNE"
 			(at 233.68 163.83 0)
 			(hide yes)
@@
 			)
 		)
-		(property "JLCPCB Part #" "C318563"
+		(property "JLCPCB Part #" "C1779"
 			(at 233.68 163.83 0)
 			(hide yes)
@@
 			)
 		)
-		(property "MPN" "RC0402FR-0710KL"
+		(property "MPN" "0402WGF1002TCE"
 			(at 226.06 113.03 0)
 			(hide yes)
@@
 			)
 		)
-		(property "JLCPCB Part #" "C60490"
+		(property "JLCPCB Part #" "C25744"
 			(at 226.06 113.03 0)
 			(hide yes)
@@
 		(body_style 1)
 		(exclude_from_sim no)
-		(in_bom yes)
+		(in_bom no)
 		(on_board yes)
 		(in_pos_files yes)
@@
 			)
 		)
-		(property "Voltage" "10V"
+		(property "Voltage" "6.3V"
 			(at 254 105.156 0)
 			(show_name no)
@@
 			)
 		)
-		(property "Voltage" "10V"
+		(property "Voltage" "6.3V"
 			(at 242.57 105.156 0)
 			(show_name no)
@@
 			)
 		)
-		(property "MPN" "RC0402FR-0718KL"
+		(property "MPN" "0402WGF1802TCE"
 			(at 196.85 120.65 0)
 			(hide yes)
@@
 			)
 		)
-		(property "JLCPCB Part #" "C138044"
+		(property "JLCPCB Part #" "C25762"
 			(at 196.85 120.65 0)
 			(hide yes)
@@
 			)
 		)
-		(property "Footprint" "Capacitor_SMD:C_0402_1005Metric"
+		(property "Footprint" "Capacitor_SMD:C_0603_1608Metric"
 			(at 187.6552 106.68 0)
 			(hide yes)
@@
 			)
 		)
-		(property "Voltage" "10V"
+		(property "Voltage" "25V"
 			(at 181.102 105.156 0)
 			(show_name no)
@@
 			)
 		)
-		(property "MPN" "CL05A106MP5NUNC"
+		(property "MPN" "CL10A106MA8NRNC"
 			(at 186.69 102.87 0)
 			(hide yes)
@@
 			)
 		)
-		(property "JLCPCB Part #" "C315248"
+		(property "JLCPCB Part #" "C96446"
 			(at 186.69 102.87 0)
 			(hide yes)
@@
 		(body_style 1)
 		(exclude_from_sim no)
-		(in_bom yes)
+		(in_bom no)
 		(on_board yes)
 		(in_pos_files yes)
